File: Hardware_Pauline/Pauline_RevB_4Layers/pauline.kicad_pcb (KiCad board)
At the start: 4 copper layers, 77.1 x 63.8 mm, 160 parts, among them J1 M20-7832046, J2 M20-7832046, J3 Wurth 61203421621, J4 Wurth 61203421621, J5 HIF3FC-10PA-2.54DSA, J6 Amphenol FCI 10129378-908001B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, J7 TE Connectivity 5-534237-2 RE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, J8 Conn_01x04_Male, Q1 BC817K-40HVL, SW1 Schurter 693-1301.9302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

Commit message: CC BY-SA 4.0 license.
git-svn-id: svn://svn.code.sf.net/p/hxcfloppyemu/code/HxCFloppyEmulator/Pauline/trunk@2084 63fa2f70-6a9b-4bc4-b855-9c6a949b1d69
Other:
- board text added: "By J-F DEL NERO (CC BY-SA 4.0)"

Commit message: Replace Nexperia/nxp 74LVC06AD buffers by standard TTL 74LS06D buffers.
git-svn-id: svn://svn.code.sf.net/p/hxcfloppyemu/code/HxCFloppyEmulator/Pauline/trunk@2145 63fa2f70-6a9b-4bc4-b855-9c6a949b1d69
Parts:
- U1, U3, U5, U7, U9: value 74LVC06AD -> SN74LS06D
Changed lines of the file:
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@@
       (effects (font (size 1 1) (thickness 0.15)) (justify mirror))
     )
-    (fp_text value 74LVC06AD (at 0 -5.28 90) (layer B.Fab)
+    (fp_text value SN74LS06D (at 0 -5.28 90) (layer B.Fab)
       (effects (font (size 1 1) (thickness 0.15)) (justify mirror))
     )
@@
       (effects (font (size 1 1) (thickness 0.15)) (justify mirror))
     )
-    (fp_text value 74LVC06AD (at 0 -5.28 90) (layer B.Fab)
+    (fp_text value SN74LS06D (at 0 -5.28 90) (layer B.Fab)
       (effects (font (size 1 1) (thickness 0.15)) (justify mirror))
     )
@@
       (effects (font (size 1 1) (thickness 0.15)) (justify mirror))
     )
-    (fp_text value 74LVC06AD (at 0 -5.28 -90) (layer B.Fab)
+    (fp_text value SN74LS06D (at 0 -5.28 -90) (layer B.Fab)
       (effects (font (size 1 1) (thickness 0.15)) (justify mirror))
     )
@@
       (effects (font (size 1 1) (thickness 0.15)) (justify mirror))
     )
-    (fp_text value 74LVC06AD (at 0 -5.28 90) (layer B.Fab)
+    (fp_text value SN74LS06D (at 0 -5.28 90) (layer B.Fab)
       (effects (font (size 1 1) (thickness 0.15)) (justify mirror))
     )
@@
       (effects (font (size 1 1) (thickness 0.15)) (justify mirror))
     )
-    (fp_text value 74LVC06AD (at 0 -5.28 -90) (layer B.Fab)
+    (fp_text value SN74LS06D (at 0 -5.28 -90) (layer B.Fab)
       (effects (font (size 1 1) (thickness 0.15)) (justify mirror))
     )

Commit message: J1,J2 reference changed to ESW-120-33-T-D.
git-svn-id: svn://svn.code.sf.net/p/hxcfloppyemu/code/HxCFloppyEmulator/Pauline/trunk@2177 63fa2f70-6a9b-4bc4-b855-9c6a949b1d69
Parts:
- J1, J2: value M20-7832046 -> ESW-120-33-T-D
Changed lines of the file:
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@@
       (effects (font (size 1 1) (thickness 0.15)) (justify mirror))
     )
-    (fp_text value M20-7832046 (at -1.27 -51.03) (layer B.Fab)
+    (fp_text value ESW-120-33-T-D (at -1.27 -51.03) (layer B.Fab)
       (effects (font (size 1 1) (thickness 0.15)) (justify mirror))
     )
@@
       (effects (font (size 1 1) (thickness 0.15)) (justify mirror))
     )
-    (fp_text value M20-7832046 (at -1.27 -51.03) (layer B.Fab)
+    (fp_text value ESW-120-33-T-D (at -1.27 -51.03) (layer B.Fab)
       (effects (font (size 1 1) (thickness 0.15)) (justify mirror))
     )
